File: ZN6_UAEFI_Adapter.kicad_sch (KiCad schematic)
At the start: 22 parts, among them J1 6376430-2, U1 ADS1015IDGS, U3 MIC5205-3.3YM5

Commit message: More Tweaks!
Parts:
- renumbered J1 to AC1
Connections:
- net FPD is gone; now on net 6_WBO1_Un: AC1.63
- net FPF is gone; now on net 5_WBO1_Rtrim: AC1.44
- net FUEL_P1 is gone; now on net GND: AC1.40
- net FUEL_P2 is gone; now on net +5VP: AC1.38
- net GNDA is gone; now on net GND: AC1.130, AC1.22, AC1.95, AC1.96, C1.2, C2.2, C3.2, C4.2, C5.2, C6.2, C7.2, C8.2, R5.1, R6.1, R7.1, R8.1, U1.1 (ADDR), U1.3 (GND), U3.2 (GND), hw-uaBrain1.B8 (GNDA), hw-uaBrain1.C6 (GNDA), hw-uaBrain1.D4 (GNDA), hw-uaBrain1.E6 (GNDA), hw-uaBrain1.E8 (GNDA), hw-uaBrain1.F5 (GNDA), hw-uaBrain1.F8 (GNDA), hw-uaBrain1.G2 (GNDA), hw-uaBrain1.J8 (GNDA), hw-uaBrain1.K6 (GNDA), hw-uaBrain1.L4 (GNDA), hw-uaBrain1.N4 (GNDA), hw-uaBrain1.P8 (GNDA)
- net IJF2 is gone; now on net 3_WBO1_Heater: AC1.62
- net IN_BUTTON1 is gone; now on net NSW: hw-uaBrain1.N7 (IN_BUTTON1)
- net IN_BUTTON2 is gone; now on net CLUTCH_SW: hw-uaBrain1.N8 (IN_BUTTON2)
- net OUT_LS6 is gone; now on net Oil_Pressure_Dash: hw-uaBrain1.L1 (OUT_LS6)
- net OUT_LS9 is gone; now on net PURGE_VALVE: hw-uaBrain1.M5 (OUT_LS9)
- net +12V: no longer AC1.37
- net +12V_RAW_FROM_ETCS: no longer hw-uaBrain1.H6 (+12V_RAW)
- net +5VP: now also AC1.36; no longer AC1.120, AC1.65, AC1.87, AC1.88
- net 1_WBO1_Ip: now also AC1.124; no longer AC1.49
- net 2_WBO1_Vm: now also AC1.115; no longer AC1.50
- net 3_WBO1_Heater: no longer AC1.52
- net 5_WBO1_Rtrim: no longer AC1.36
- net 6_WBO1_Un: no longer AC1.39
- net CLUTCH_SW: no longer hw-uaBrain1.K4 (IN_HALL3)
- net FUEL_PRESSURE: now also AC1.56; no longer AC1.29
- net GND: now also AC1.28, AC1.45, AC1.65; no longer AC1.104
- net IN_FLEX: now also AC1.25; no longer AC1.45
- net IN_IAT: now also AC1.52; no longer AC1.12
- net IN_KNOCK1_RAW: now also AC1.48; no longer AC1.59
- net IN_KNOCK2_RAW: now also AC1.59; no longer AC1.48
- net IN_TPS1: now also AC1.49; no longer AC1.129
- net IN_TPS2: now also AC1.50; no longer AC1.119
- net OIL_PRESSURE: now also AC1.117; no longer AC1.56
- net OUT_DC1+: now also AC1.119; no longer AC1.102
- net OUT_DC1-: now also AC1.120; no longer AC1.103
- net OUT_DC2+: now also AC1.102; no longer AC1.106
- net OUT_DC2-: now also AC1.103; no longer AC1.107
- net OUT_IGN1: now also AC1.122; no longer AC1.109
- net OUT_IGN2: now also AC1.111; no longer AC1.132
- net OUT_IGN3: now also AC1.132; no longer AC1.133
- net OUT_IGN4: now also AC1.109; no longer AC1.111
- net OUT_IGN5: now also AC1.129; no longer AC1.126
- net OUT_IGN6: now also AC1.106; no longer AC1.122
- net OUT_INJ2: now also AC1.123; no longer AC1.114
- net OUT_INJ3: now also AC1.133; no longer AC1.115
- net OUT_INJ4: now also AC1.114; no longer AC1.123
- net OUT_INJ5: now also AC1.107; no longer AC1.124
- net OUT_INJ6: now also AC1.108; no longer AC1.125
- net EGT1-: now reaches hw-uaBrain1.A7 (EGT1-)
- net EGT1-: now also AC1.125
- net EGT1+: now reaches hw-uaBrain1.A8 (EGT1+)
- net EGT1+: now also AC1.126
- net Oil_Pressure_Dash: now reaches AC1.31
- net AC: no longer names the net of AC1.101
- net ACP: no longer names the net of AC1.8
- net A/C Clutch: no longer names the net of AC1.66
- net BLOWER_HB: no longer names the net of AC1.20
- net EGT2+: no longer names the net of hw-uaBrain1.H8 (EGT2+)
- net EGT2-: no longer names the net of hw-uaBrain1.H7 (EGT2-)
- net IJF1: no longer names the net of AC1.42
- net IMO: no longer names the net of AC1.91
- net IN_HALL1 renamed VVT Inlet Sensor RH
- net IN_HALL2 renamed VVT Inlet Sensor LH
- net LIN_ALTERNATOR: no longer names the net of AC1.21
- net OUT_LS10: no longer names the net of hw-uaBrain1.M6 (OUT_LS10)
- net SHIELD: no longer names the net of AC1.61
- net SHIELD: no longer AC1.28
- net ST1-: no longer names the net of AC1.3
- net STAR: no longer names the net of AC1.100
- net STARTER: no longer names the net of AC1.92
- net STSW2+1: no longer names the net of AC1.14
- net STSW2+2: no longer names the net of AC1.17
- net TACH: no longer names the net of AC1.81
- net VVT Inlet Bank 1 renamed VVT Inlet Solenoid LH
- net VVT Inlet Solenoid LH: now also hw-uaBrain1.M8 (OUT_LS2); no longer hw-uaBrain1.M7 (OUT_LS1)
- removed net VVT Inlet Bank 2: AC1.117, hw-uaBrain1.M8 (OUT_LS2)
- net WFSE: no longer names the net of AC1.43
- new net VVT Inlet Solenoid RH: AC1.39, hw-uaBrain1.M7 (OUT_LS1)
- no-connect marks 49 -> 52

Commit message: First Draft of Adapter board
Parts:
- removed C1: 1uF, Capacitor_SMD:C_0603_1608Metric, symbol Device:C_Small
- removed C2, C3, C4, C5: 10nF, Capacitor_SMD:C_0603_1608Metric, symbol Device:C_Small
- removed R1, R2, R3, R4: 10k, Resistor_SMD:R_0603_1608Metric, symbol Device:R_Small
- removed R5, R6, R7, R8: 20k, Resistor_SMD:R_0603_1608Metric, symbol Device:R_Small
- removed U1: ADS1015IDGS, Package_SO:TSSOP-10_3x3mm_P0.5mm, symbol Analog_ADC:ADS1015IDGS
- added AC2: 6376430-2, ZN6:TE_6376430-2, symbol ZN6_Adapter:6376430-2
- added D2, D3, D4: SMBJ24A, Diode_SMD:D_SMB, symbol Device:D_Zener_Small
- added D5: SZNUP2105L, Package_TO_SOT_SMD:SOT-23, symbol Power_Protection:SZNUP2105L
- added J1, J2: Conn_01x32_Socket, Connector_PinHeader_2.54mm:PinHeader_1x32_P2.54mm_Vertical, symbol Connector:Conn_01x32_Socket
- added J12, J13, J14: Conn_01x06_Socket, Connector_PinHeader_2.54mm:PinHeader_1x06_P2.54mm_Vertical, symbol Connector:Conn_01x06_Socket
- added J3: Conn_01x02_Socket, Connector_PinHeader_2.54mm:PinHeader_1x02_P2.54mm_Vertical, symbol Connector:Conn_01x02_Socket
- added J4, J5: Conn_01x24_Socket, Connector_PinHeader_2.54mm:PinHeader_1x24_P2.54mm_Vertical, symbol Connector:Conn_01x24_Socket
Connections:
- net +12V: now also AC2.1, D2.1 (K), J2.9 (Pin_9)
- net +12V_CONSTANT: now also AC2.2, D4.1 (K)
- net +3.3VA: now also J2.5 (Pin_5); no longer hw-uaBrain1.D5 (+3.3VA)
- net 12V_KEY: now also AC2.27, D3.1 (K), J2.10 (Pin_10)
- net CAN1+: now also AC2.19, D5.1 (K), J2.21 (Pin_21)
- net CAN1-: now also AC2.18, D5.2 (K), J2.22 (Pin_22)
- net GND: now also AC1.104, AC1.4, AC1.60, AC1.61, AC1.66, AC2.104, AC2.105, AC2.28, AC2.32, AC2.33, AC2.34, AC2.4, AC2.60, AC2.61, AC2.66, D2.2 (A), D3.2 (A), D4.2 (A), D5.3 (A), J1.19 (Pin_19), J1.24 (Pin_24), J2.11 (Pin_11), J2.12 (Pin_12), J2.29 (Pin_29), J4.24 (Pin_24), J5.19 (Pin_19), J5.24 (Pin_24); no longer AC1.130, AC1.22, AC1.40, AC1.45, AC1.65, AC1.95, AC1.96, C6.2, C7.2, C8.2, U3.2 (GND), hw-uaBrain1.B8 (GNDA), hw-uaBrain1.C6 (GNDA), hw-uaBrain1.D4 (GNDA), hw-uaBrain1.E6 (GNDA), hw-uaBrain1.E8 (GNDA), hw-uaBrain1.F5 (GNDA), hw-uaBrain1.F8 (GNDA), hw-uaBrain1.G2 (GNDA), hw-uaBrain1.J8 (GNDA), hw-uaBrain1.K6 (GNDA), hw-uaBrain1.L4 (GNDA), hw-uaBrain1.N4 (GNDA), hw-uaBrain1.P8 (GNDA)
- net SCL: now also J2.8 (Pin_8)
- net SDA: now also J2.6 (Pin_6)
- net at AC1.100: now also AC2.100
- net at AC1.101: now also AC2.101
- net at AC1.67: now also AC2.67
- net at AC1.68: now also AC2.68
- net at AC1.69: now also AC2.69
- net at AC1.70: now also AC2.70
- net at AC1.72: now also AC2.72
- net at AC1.74: now also AC2.74
- net at AC1.75: now also AC2.75
- net at AC1.80: now also AC2.80
- net at AC1.81: now also AC2.81
- net at AC1.82: now also AC2.82
- net at AC1.84: now also AC2.84
- net at AC1.86: now also AC2.86
- net at AC1.87: now also AC2.87
- net at AC1.88: now also AC2.88
- net at AC1.90: now also AC2.90
- net at AC1.91: now also AC2.91
- net at AC1.92: now also AC2.92
- net at AC1.93: now also AC2.93
- net at AC1.94: now also AC2.94
- net at AC1.98: now also AC2.98
- net at AC1.99: now also AC2.99
- net at hw-uaBrain1.C1 (VR_DISCRETE-): now also J1.17 (Pin_17)
- net at hw-uaBrain1.C2 (VR_DISCRETE+): now also J1.18 (Pin_18)
- net at hw-uaBrain1.D2 (IN_AUX1): now also J1.26 (Pin_26)
- net at hw-uaBrain1.F3 (IN_AUX2): now also J4.11 (Pin_11)
- net at hw-uaBrain1.G4 (CAN2+): now also J4.20 (Pin_20)
- net at hw-uaBrain1.G5 (CAN2-): now also J4.21 (Pin_21)
- net at hw-uaBrain1.H1 (6_WBO2_Un): now also J5.1 (Pin_1)
- net at hw-uaBrain1.H2 (5_WBO2_Rtrim): now also J5.2 (Pin_2)
- net at hw-uaBrain1.H3 (1_WBO2_Ip): now also J5.3 (Pin_3)
- net at hw-uaBrain1.H4 (2_WBO2_Vm): now also J5.4 (Pin_4)
- net at hw-uaBrain1.H5 (3_WBO2_Heater): now also J5.5 (Pin_5)
- net at hw-uaBrain1.H6 (+12V_RAW): now also J5.6 (Pin_6)
- net at hw-uaBrain1.H7 (EGT2-): now also J5.7 (Pin_7)
- net at hw-uaBrain1.H8 (EGT2+): now also J5.8 (Pin_8)
- net at hw-uaBrain1.K4 (IN_HALL3): now also J5.20 (Pin_20)
- net at AC1.35: now also AC2.35
- net at AC1.37: now also AC2.37
- net at AC1.41: now also AC2.41
- net at AC1.42: now also AC2.42
- net at AC1.43: now also AC2.43
- net at AC1.53: now also AC2.53
- net at AC1.54: now also AC2.54
- net at AC1.55: now also AC2.55
- net at AC1.64: now also AC2.64
- net at AC1.10: now also AC2.10
- net at AC1.11: now also AC2.11
- net at AC1.12: now also AC2.12
- net at AC1.13: now also AC2.13
- net at AC1.14: now also AC2.14
- net at AC1.17: now also AC2.17
- net at AC1.20: now also AC2.20
- net at AC1.21: now also AC2.21
- net at AC1.23: now also AC2.23
- net at AC1.24: now also AC2.24
- net at AC1.26: now also AC2.26
- net at AC1.29: now also AC2.29
- net at AC1.3: now also AC2.3
- net at AC1.5: now also AC2.5
- net at AC1.6: now also AC2.6
- net at AC1.8: now also AC2.8
- net at AC1.9: now also AC2.9
- net at AC1.110: now also AC2.110
- net at AC1.116: now also AC2.116
- net at AC1.127: now also AC2.127
- net at AC1.128: now also AC2.128
- net at AC1.134: now also AC2.134
- net at AC1.135: now also AC2.135
- net at hw-uaBrain1.M6 (OUT_LS10): now also J2.14 (Pin_14)
- net at hw-uaBrain1.P1 (PROG_BUTTON): now also J2.25 (Pin_25)
- net at hw-uaBrain1.P2 (VBUS): now also J2.26 (Pin_26)
- net at hw-uaBrain1.P3 (USB-): now also J2.27 (Pin_27)
- net at hw-uaBrain1.P4 (USB+): now also J2.28 (Pin_28)
- net +12V_RAW_FROM_ETCS: no longer names the net of AC1.73
- net +12V_RAW_FROM_ETCS: now also AC2.73; no longer hw-uaBrain1.A6 (+12V_RAW)
- net +3.3V: no longer names the net of hw-uaBrain1.D6 (+3.3V)
- net +3.3V: now also J1.30 (Pin_30)
- net +5V: no longer names the net of hw-uaBrain1.D8 (+5V)
- net +5V: now also J1.32 (Pin_32)
- net +5VA: no longer names the net of hw-uaBrain1.L7 (+5VA)
- net +5VA: now also J2.7 (Pin_7); no longer hw-uaBrain1.D7 (+5VA)
- removed net +5VP: AC1.36, AC1.38, hw-uaBrain1.C5 (+5VP), hw-uaBrain1.D3 (+5VP), hw-uaBrain1.E5 (+5VP), hw-uaBrain1.F4 (+5VP), hw-uaBrain1.F7 (+5VP), hw-uaBrain1.K5 (+5VP), hw-uaBrain1.L3 (+5VP), hw-uaBrain1.N3 (+5VP), hw-uaBrain1.P7 (+5VP)
- net 1_WBO1_Ip: no longer names the net of hw-uaBrain1.A3 (1_WBO1_Ip)
- net 1_WBO1_Ip: now also J1.3 (Pin_3); no longer AC1.124
- net 2_WBO1_Vm: no longer names the net of hw-uaBrain1.A4 (2_WBO1_Vm)
- net 2_WBO1_Vm: now also J1.4 (Pin_4); no longer AC1.115
- net 3_WBO1_Heater: no longer names the net of hw-uaBrain1.A5 (3_WBO1_Heater)
- net 3_WBO1_Heater: now also J1.5 (Pin_5); no longer AC1.62
- net 5_WBO1_Rtrim: no longer names the net of hw-uaBrain1.A2 (5_WBO1_Rtrim)
- net 5_WBO1_Rtrim: now also J1.2 (Pin_2); no longer AC1.44
- net 6_WBO1_Un: no longer names the net of hw-uaBrain1.A1 (6_WBO1_Un)
- net 6_WBO1_Un: now also J1.1 (Pin_1); no longer AC1.63
- net BRAKE_SW: no longer names the net of AC1.7
- net BRAKE_SW: now also AC2.7
- net CLUTCH_SW: no longer names the net of hw-uaBrain1.N8 (IN_BUTTON2)
- net CLUTCH_SW: now also J2.24 (Pin_24); no longer AC1.15
- net CRANK_VR+: no longer names the net of hw-uaBrain1.K2 (VR_MAX9924+)
- net CRANK_VR+: now also J5.18 (Pin_18); no longer AC1.47
- net CRANK_VR-: no longer names the net of hw-uaBrain1.K1 (VR_MAX9924-)
- net CRANK_VR-: now also J5.17 (Pin_17); no longer AC1.58
- net CRUISE_CCS: no longer names the net of AC1.30
- net CRUISE_CCS: now also AC2.30
- net EFI_RELAYS: no longer names the net of AC1.79
- net EFI_RELAYS: now also AC2.79
- net EGT1+: no longer names the net of hw-uaBrain1.A8 (EGT1+)
- net EGT1+: now also J1.8 (Pin_8); no longer AC1.126
- net EGT1-: no longer names the net of hw-uaBrain1.A7 (EGT1-)
- net EGT1-: now also J1.7 (Pin_7); no longer AC1.125
- removed net ETCS_RELAY: AC1.71, AC1.76, AC1.83, hw-uaBrain1.C7 (OUT_LS3)
- net FAN1: no longer names the net of AC1.77
- net FAN1: now also AC2.77; no longer hw-uaBrain1.G6 (OUT_LS7)
- net FAN2: no longer names the net of AC1.78
- net FAN2: now also AC2.78; no longer hw-uaBrain1.G7 (OUT_LS8)
- net FP_CONTROL: no longer names the net of AC1.85
- net FP_CONTROL: now also AC2.85; no longer hw-uaBrain1.D1 (OUT_LS4)
- net FUEL_PRESSURE: no longer names the net of AC1.56
- net FUEL_PRESSURE: now also AC2.56
- net IN_BUTTON3: no longer names the net of hw-uaBrain1.L2 (IN_BUTTON3)
- net IN_BUTTON3: now also J2.2 (Pin_2)
- net IN_CLT: no longer names the net of hw-uaBrain1.E7 (IN_CLT)
- net IN_CLT: now also J4.7 (Pin_7); no longer AC1.131
- net IN_FLEX: no longer names the net of hw-uaBrain1.P6 (IN_FLEX)
- net IN_FLEX: now also J2.30 (Pin_30); no longer AC1.25
- net IN_IAT: no longer names the net of hw-uaBrain1.G1 (IN_IAT)
- net IN_IAT: now also J4.17 (Pin_17); no longer AC1.52
- net IN_KNOCK1_RAW: no longer names the net of hw-uaBrain1.B7 (IN_KNOCK1_RAW)
- net IN_KNOCK1_RAW: now also J1.15 (Pin_15); no longer AC1.48
- net IN_KNOCK2_RAW: no longer names the net of hw-uaBrain1.J7 (IN_KNOCK2_RAW)
- net IN_KNOCK2_RAW: now also J5.15 (Pin_15); no longer AC1.59
- net IN_MAP: no longer names the net of hw-uaBrain1.F6 (IN_MAP)
- net IN_MAP: now also J4.14 (Pin_14); no longer AC1.51
- net IN_PPS1: no longer names the net of AC1.89
- net IN_PPS1: now also AC2.89; no longer hw-uaBrain1.N1 (IN_PPS1)
- net IN_PPS2: no longer names the net of AC1.97
- net IN_PPS2: now also AC2.97; no longer hw-uaBrain1.N2 (IN_PPS2)
- net IN_TPS1: no longer names the net of hw-uaBrain1.E3 (IN_TPS1)
- net IN_TPS1: now also J4.3 (Pin_3); no longer AC1.49
- net IN_TPS2: no longer names the net of hw-uaBrain1.E4 (IN_TPS2)
- net IN_TPS2: now also J4.4 (Pin_4); no longer AC1.50
- net NSW: no longer names the net of hw-uaBrain1.N7 (IN_BUTTON1)
- net NSW: now also J2.23 (Pin_23); no longer AC1.16
- net OIL_PRESSURE: no longer names the net of AC1.117
- net OIL_PRESSURE: now also AC2.117
- net OIL_TEMP: no longer names the net of AC1.121
- net OIL_TEMP: now also AC2.121
- net OUT_DC1+: no longer names the net of hw-uaBrain1.E2 (OUT_DC1+)
- net OUT_DC1+: now also J4.2 (Pin_2); no longer AC1.119
- net OUT_DC1-: no longer names the net of hw-uaBrain1.E1 (OUT_DC1-)
- net OUT_DC1-: now also J4.1 (Pin_1); no longer AC1.120
- net OUT_DC2+: no longer names the net of hw-uaBrain1.F2 (OUT_DC2+)
- net OUT_DC2+: now also J4.10 (Pin_10); no longer AC1.102
- net OUT_DC2-: no longer names the net of hw-uaBrain1.F1 (OUT_DC2-)
- net OUT_DC2-: now also J4.9 (Pin_9); no longer AC1.103
- net OUT_IGN1: no longer names the net of hw-uaBrain1.B1 (OUT_IGN1)
- net OUT_IGN1: now also J1.9 (Pin_9); no longer AC1.122
- net OUT_IGN2: no longer names the net of hw-uaBrain1.B2 (OUT_IGN2)
- net OUT_IGN2: now also J1.10 (Pin_10); no longer AC1.111
- net OUT_IGN3: no longer names the net of hw-uaBrain1.B3 (OUT_IGN3)
- net OUT_IGN3: now also J1.11 (Pin_11); no longer AC1.132
- net OUT_IGN4: no longer names the net of hw-uaBrain1.J1 (OUT_IGN4)
- net OUT_IGN4: now also J5.9 (Pin_9); no longer AC1.109
- net OUT_IGN5: no longer names the net of hw-uaBrain1.J2 (OUT_IGN5)
- net OUT_IGN5: now also J5.10 (Pin_10); no longer AC1.129
- net OUT_IGN6: no longer names the net of hw-uaBrain1.J3 (OUT_IGN6)
- net OUT_IGN6: now also J5.11 (Pin_11); no longer AC1.106
- net OUT_INJ1: no longer names the net of hw-uaBrain1.B4 (OUT_INJ1)
- net OUT_INJ1: now also J1.12 (Pin_12); no longer AC1.113
- net OUT_INJ2: no longer names the net of hw-uaBrain1.B5 (OUT_INJ2)
- net OUT_INJ2: now also J1.13 (Pin_13); no longer AC1.123
- net OUT_INJ3: no longer names the net of hw-uaBrain1.B6 (OUT_INJ3)
- net OUT_INJ3: now also J1.14 (Pin_14); no longer AC1.133
- net OUT_INJ4: no longer names the net of hw-uaBrain1.J4 (OUT_INJ4)
- net OUT_INJ4: now also J5.12 (Pin_12); no longer AC1.114
- net OUT_INJ5: no longer names the net of hw-uaBrain1.J5 (OUT_INJ5)
- net OUT_INJ5: now also J5.13 (Pin_13); no longer AC1.107
- net OUT_INJ6: no longer names the net of hw-uaBrain1.J6 (OUT_INJ6)
- net OUT_INJ6: now also J5.14 (Pin_14); no longer AC1.108
- net OUT_LS5: no longer names the net of hw-uaBrain1.K7 (OUT_LS5)
- net OUT_LS5: now also J5.23 (Pin_23)
- net Oil_Pressure_Dash: no longer names the net of hw-uaBrain1.L1 (OUT_LS6)
- net Oil_Pressure_Dash: now also J2.1 (Pin_1); no longer AC1.31
- net PURGE_VALVE: no longer names the net of hw-uaBrain1.M5 (OUT_LS9)
- net PURGE_VALVE: now also J2.13 (Pin_13); no longer AC1.112
- net VVT Inlet Sensor LH: no longer names the net of hw-uaBrain1.G3 (IN_HALL2)
- net VVT Inlet Sensor LH: now also J4.19 (Pin_19); no longer AC1.46
- net VVT Inlet Sensor RH: no longer names the net of hw-uaBrain1.C4 (IN_HALL1)
- net VVT Inlet Sensor RH: now also J1.20 (Pin_20); no longer AC1.57
- net VVT Inlet Solenoid LH: no longer names the net of hw-uaBrain1.M8 (OUT_LS2)
- net VVT Inlet Solenoid LH: now also J2.16 (Pin_16); no longer AC1.118
- net VVT Inlet Solenoid RH: no longer names the net of hw-uaBrain1.M7 (OUT_LS1)
- net VVT Inlet Solenoid RH: now also J2.15 (Pin_15); no longer AC1.39
- new net: AC1.71, AC2.71
- new net: AC1.76, AC2.76
- new net: AC1.83, AC2.83
- new net: AC1.95, AC2.95
- new net: AC1.96, AC2.96
- new net: J4.12 (Pin_12), hw-uaBrain1.F4 (+5VP)
- new net: J4.13 (Pin_13), hw-uaBrain1.F5 (GNDA)
- new net: J4.15 (Pin_15), hw-uaBrain1.F7 (+5VP)
- new net: J4.16 (Pin_16), hw-uaBrain1.F8 (GNDA)
- new net: J4.18 (Pin_18), hw-uaBrain1.G2 (GNDA)
- new net: J4.22 (Pin_22), hw-uaBrain1.G6 (OUT_LS7)
- new net: J4.23 (Pin_23), hw-uaBrain1.G7 (OUT_LS8)
- new net: J4.5 (Pin_5), hw-uaBrain1.E5 (+5VP)
- new net: J4.6 (Pin_6), hw-uaBrain1.E6 (GNDA)
- new net: J4.8 (Pin_8), hw-uaBrain1.E8 (GNDA)
- new net: J2.17 (Pin_17), hw-uaBrain1.N1 (IN_PPS1)
- new net: J2.18 (Pin_18), hw-uaBrain1.N2 (IN_PPS2)
- new net: J2.19 (Pin_19), hw-uaBrain1.N3 (+5VP)
- new net: J2.20 (Pin_20), hw-uaBrain1.N4 (GNDA)
- new net: J2.31 (Pin_31), hw-uaBrain1.P7 (+5VP)
- new net: J2.32 (Pin_32), hw-uaBrain1.P8 (GNDA)
- new net: AC1.15, AC2.15
- new net: AC1.16, AC2.16
- new net: AC1.22, AC2.22
- new net: AC1.25, AC2.25
- new net: AC1.31, AC2.31
- new net: J1.16 (Pin_16), hw-uaBrain1.B8 (GNDA)
- new net: J1.21 (Pin_21), hw-uaBrain1.C5 (+5VP)
- new net: J1.22 (Pin_22), hw-uaBrain1.C6 (GNDA)
- new net: J1.23 (Pin_23), hw-uaBrain1.C7 (OUT_LS3)
- new net: J1.25 (Pin_25), hw-uaBrain1.D1 (OUT_LS4)
- new net: J1.27 (Pin_27), hw-uaBrain1.D3 (+5VP)
- new net: J1.28 (Pin_28), hw-uaBrain1.D4 (GNDA)
- new net: J1.29 (Pin_29), hw-uaBrain1.D5 (+3.3VA)
- new net: J1.31 (Pin_31), hw-uaBrain1.D7 (+5VA)
- new net: J1.6 (Pin_6), hw-uaBrain1.A6 (+12V_RAW)
- new net: J5.16 (Pin_16), hw-uaBrain1.J8 (GNDA)
- new net: J5.21 (Pin_21), hw-uaBrain1.K5 (+5VP)
- new net: J5.22 (Pin_22), hw-uaBrain1.K6 (GNDA)
- new net: AC1.36, AC2.36
- new net: AC1.38, AC2.38
- new net: AC1.39, AC2.39
- new net: AC1.40, AC2.40
- new net: AC1.44, AC2.44
- new net: AC1.45, AC2.45
- new net: AC1.46, AC2.46
- new net: AC1.47, AC2.47
- new net: AC1.48, AC2.48
- new net: AC1.49, AC2.49
- new net: AC1.50, AC2.50
- new net: AC1.51, AC2.51
- new net: AC1.52, AC2.52
- new net: AC1.57, AC2.57
- new net: AC1.58, AC2.58
- new net: AC1.59, AC2.59
- new net: AC1.62, AC2.62
- new net: AC1.63, AC2.63
- new net: AC1.65, AC2.65
- new net: AC1.102, AC2.102
- new net: AC1.103, AC2.103
- new net: AC1.106, AC2.106
- new net: AC1.107, AC2.107
- new net: AC1.108, AC2.108
- new net: AC1.109, AC2.109
- new net: AC1.111, AC2.111
- new net: AC1.112, AC2.112
- new net: AC1.113, AC2.113
- new net: AC1.114, AC2.114
- new net: AC1.115, AC2.115
- new net: AC1.118, AC2.118
- new net: AC1.119, AC2.119
- new net: AC1.120, AC2.120
- new net: AC1.122, AC2.122
- new net: AC1.123, AC2.123
- new net: AC1.124, AC2.124
- new net: AC1.125, AC2.125
- new net: AC1.126, AC2.126
- new net: AC1.129, AC2.129
- new net: AC1.130, AC2.130
- new net: AC1.131, AC2.131
- new net: AC1.132, AC2.132
- new net: AC1.133, AC2.133
- new net 5VP: J14.1 (Pin_1), J14.2 (Pin_2), J14.3 (Pin_3), J14.4 (Pin_4), J14.5 (Pin_5), J14.6 (Pin_6), J2.3 (Pin_3), hw-uaBrain1.L3 (+5VP)
- new net ADS712/EXPADIN_0: J13.1 (Pin_1)
- new net ADS712/EXPADIN_1: J13.2 (Pin_2)
- new net ADS712/EXPADIN_2: J13.3 (Pin_3)
- new net ADS712/EXPADIN_3: J13.4 (Pin_4)
- new net ADS712/EXPADIN_4: J13.5 (Pin_5)
- new net ADS712/EXPADIN_5: J13.6 (Pin_6)
- new net ADS712/LS_AUX_1: J3.1 (Pin_1)
- new net ADS712/LS_AUX_2: J3.2 (Pin_2)
- new net GNDA: C6.2, C7.2, C8.2, J12.1 (Pin_1), J12.2 (Pin_2), J12.3 (Pin_3), J12.4 (Pin_4), J12.5 (Pin_5), J12.6 (Pin_6), J2.4 (Pin_4), U3.2 (GND), hw-uaBrain1.L4 (GNDA)
- no-connect marks 52 -> 1
Other:
- added sheet ADS712 (ADS712.kicad_sch)
- note added: "8CH IO Expansion"
- note added: "ESD"
- note added: "Inputs x6 10k Pullup to 5V Analog or Digital Low Speed Low Side Outputs 42V 2A+ Short−Circuit Protection Thermal Shutdown with Automatic Restart Overvoltage Protection Integrated Clamp for Inductive Switching"
- note removed: "0x24"
- note removed: "ETCS Relay Repurposes for O2 Heaters through ECU"
- note removed: "EXTRA ANALOG"
- moved on the sheet: hw-uaBrain1A

Commit message: Re-adjust project for uaEFI instead.
Parts:
- removed C6, C7: 1uF, Capacitor_SMD:C_0603_1608Metric, symbol Device:C_Small
- removed C8: 10uF, Capacitor_SMD:C_0603_1608Metric, symbol Device:C_Small
- removed D1: 1N4148WS, Diode_SMD:D_SOD-323F, symbol Device:D_Small
- removed D2, D3, D4: SMBJ24A, Diode_SMD:D_SMB, symbol Device:D_Zener_Small
- removed D5: SZNUP2105L, Package_TO_SOT_SMD:SOT-23, symbol Power_Protection:SZNUP2105L
- removed J1, J2: Conn_01x32_Socket, Connector_PinHeader_2.54mm:PinHeader_1x32_P2.54mm_Vertical, symbol Connector:Conn_01x32_Socket
- removed J12, J13, J14: Conn_01x06_Socket, Connector_PinHeader_2.54mm:PinHeader_1x06_P2.54mm_Vertical, symbol Connector:Conn_01x06_Socket
- removed J3: Conn_01x02_Socket, Connector_PinHeader_2.54mm:PinHeader_1x02_P2.54mm_Vertical, symbol Connector:Conn_01x02_Socket
- removed J4, J5: Conn_01x24_Socket, Connector_PinHeader_2.54mm:PinHeader_1x24_P2.54mm_Vertical, symbol Connector:Conn_01x24_Socket
- removed TP1: VBAT, Connector_PinHeader_2.54mm:PinHeader_1x01_P2.54mm_Vertical, symbol Connector:TestPoint
- removed U3: MIC5205-3.3YM5, Package_TO_SOT_SMD:SOT-23-5, symbol Regulator_Linear:MIC5205-3.3YM5
- removed hw-uaBrain1: hw-uaBrain, ZN6:hw-uaBrain, symbol ZN6_Adapter:hw-uaBrain
- added H1, H2, H3, H4: MountingHole, MountingHole:MountingHole_3.2mm_M3, symbol Mechanical:MountingHole
- added J1, J2, J3, J4, J5, J6: Conn_01x04_Socket, Connector_PinHeader_2.54mm:PinHeader_1x04_P2.54mm_Vertical, symbol Connector:Conn_01x04_Socket
Connections:
- net GND: now also J3.1 (Pin_1), J3.2 (Pin_2), J3.3 (Pin_3), J3.4 (Pin_4)
- net +12V: no longer names the net of AC1.1, AC2.1
- net +12V_CONSTANT: no longer names the net of AC1.2, AC2.2
- net 12V_KEY: no longer names the net of AC1.27, AC2.27
- new net: J2.1 (Pin_1), J2.2 (Pin_2), J2.3 (Pin_3), J2.4 (Pin_4)
- new net: J1.1 (Pin_1), J1.2 (Pin_2), J1.3 (Pin_3), J1.4 (Pin_4)
- no-connect marks 1 -> 0
Other:
- removed sheet ADS712
- note added: "UAEFI"
- note removed: "8CH IO Expansion"
- note removed: "ESD"
- note removed: "Inputs x6 10k Pullup to 5V Analog or Digital Low Speed Low Side Outputs 42V 2A+ Short−Circuit Protection Thermal Shutdown with Automatic Restart Overvoltage Protection Integrated Clamp for Inductive Switching"
- note removed: "UAEFI BRAIN"
- note removed: "Use Jumper Wire to Brain bat"
- note removed: "VBAT POWER"
- moved on the sheet: AC1A, AC1B, AC1C, AC1D, AC2A, AC2B, AC2C, AC2D
