File: ZN6_ATLAS_Adapter.kicad_pcb (KiCad board)
At the start: 4 copper layers, 170 x 114 mm, 72 parts, among them J1 Conn_01x04_Socket, J2 Conn_01x04_Socket, J3 Conn_01x04_Socket, J4 Conn_01x04_Socket, J5 Conn_01x04_Socket, J6 Conn_01x04_Socket, J7 Conn_01x02_Socket, J8 Conn_01x04_Socket, J9 Conn_01x05_Pin, M1 Polygonus ECU Module, M2 Polygonus ECU Module, U2 TLE9201SG, U25 MAX9924, U3 TLE9201SG, U4 VNLD5090, U5 VNLD5090, U6 LSM6DSV

Commit message: Add TVS protection and clarify board nets
Add SMAJ36A protection to the 12V rails and ETCS input, label adapter signal nets, update routing, and document the hard-wired ECU pins.
Parts:
- added D1: SMAJ36A, Diode_SMD:D_SMA, F.Cu at (104.3, 84.4)
- added D2: SMAJ36A, Diode_SMD:D_SMA, F.Cu at (104.3, 109.1)
- added D3: SMAJ36A, Diode_SMD:D_SMA, F.Cu at (105.1, 151.8)
- added D4: SMAJ36A, Diode_SMD:D_SMA, F.Cu at (122.2, 160.4)
- moved R10 0.45 mm to (156.2, 95.0)
- moved C35 0.20 mm to (137.5, 160.4)
Connections:
- net Net-(M1-IGN10) renamed /IGN10
- net Net-(M1-IGN11) renamed /IGN11
- net Net-(M1-IGN12) renamed /IGN12
- net Net-(M1-Knock_1) renamed /KNOCK1
- net Net-(M1-Knock_2) renamed /KNOCK2
- net Net-(M1-LS1) renamed /LS1
- net Net-(M1-LS2) renamed /LS2
- net Net-(M1-LS3) renamed /LS3
- net Net-(M1-LS4) renamed /LS4
- net Net-(M1-LS5) renamed /LS5
- net Net-(M1-LS6) renamed /LS6
- net Net-(M1-LS7) renamed /LS7
- net Net-(M1-LS8) renamed /LS8
- net Net-(M1-RC1) renamed /RC1
- net Net-(M1-RC2) renamed /RC2
- net Net-(M1-VR2) renamed /VR2
- AC1 pad 4: GND -> Net-(AC1-Pad4)
- AC2 pad 4: GND -> Net-(AC1-Pad4)
- M1 pad 32: Net-(M1-12V_MR-Pad32) -> /12V_MR
- M2 pad 32: Net-(M1-12V_MR-Pad32) -> /12V_MR
Routing:
- net /12V_MR: track 76.6 -> 162.3 mm
- net /ETCS: track 137.9 -> 193.7 mm
- net Net-(AC1-Pad4): track 0.00 -> 28.4 mm
- net GND: track 9.86 -> 2.24 mm, vias 171 -> 182
- net Net-(M1-12V_MR-Pad32): track 7.00 -> 0.00 mm
- net /DC2_DIS: track 18.7 -> 17.7 mm
Other:
- board text added: "GND GND"
