File: ZN6_ATLAS_Adapter.kicad_sch (KiCad schematic)
At the start: 40 parts, among them J1 Conn_01x04_Socket, J2 Conn_01x04_Socket, J3 Conn_01x04_Socket, J4 Conn_01x04_Socket, J5 Conn_01x04_Socket, J6 Conn_01x04_Socket, J7 Conn_01x02_Socket, J8 Conn_01x04_Socket, J9 Conn_01x05_Pin, M1 Polygonus ECU Module, M2 Polygonus ECU Module, U25 MAX9924, U4 VNLD5090, U5 VNLD5090, U6 LSM6DSV

Commit message: Add TVS protection and clarify board nets
Add SMAJ36A protection to the 12V rails and ETCS input, label adapter signal nets, update routing, and document the hard-wired ECU pins.
Parts:
- added D1, D2, D3, D4: SMAJ36A, Diode_SMD:D_SMA, symbol Device:D_Zener_Small
Connections:
- net 12V_Constant: now also D3.1 (K)
- net 12V_MR: now also M1.32 (12V_MR), M2.32 (12V_MR), D4.1 (K)
- net 12V_SW: now also D2.1 (K)
- net ETCS: now also D1.1 (K)
- net GND: now also D1.2 (A), D2.2 (A), D3.2 (A), D4.2 (A); no longer AC1.4, AC2.4
- net LS7: now reaches M1.10 (LS7), M2.10 (LS7)
- net LS8: now reaches M1.11 (LS8), M2.11 (LS8)
- net IGN12: now reaches M1.12 (IGN12), M2.12 (IGN12)
- net IGN11: now reaches M1.13 (IGN11), M2.13 (IGN11)
- net IGN10: now reaches M1.14 (IGN10), M2.14 (IGN10)
- net LS1: now reaches M1.4 (LS1), M2.4 (LS1)
- net LS2: now reaches M1.5 (LS2), M2.5 (LS2)
- net LS3: now reaches M1.6 (LS3), M2.6 (LS3)
- net KNOCK1: now reaches M1.63 (Knock_1), M2.63 (Knock_1)
- net KNOCK2: now reaches M1.64 (Knock_2), M2.64 (Knock_2)
- net LS4: now reaches M1.7 (LS4), M2.7 (LS4)
- net RC1: now reaches M1.75 (RC1), M2.75 (RC1)
- net RC2: now reaches M1.76 (RC2), M2.76 (RC2)
- net LS5: now reaches M1.8 (LS5), M2.8 (LS5)
- net LS6: now reaches M1.9 (LS6), M2.9 (LS6)
- net VR2: now reaches M1.95 (VR2), M2.95 (VR2)
- new net: AC1.4, AC2.4
Other:
- moved on the sheet: C35, C40, J9
